Commit message: generating points for each leg in tip trajectory generator node. still have to be transformed to body frame and still nothing is tested yet

File: install/hexapod_description/share/hexapod_description/urdf/hexapod.urdf.xacro (robot description, xacro)
@@ -702,3 +702,20 @@
         <child link="e6" />
     </joint>
+    <!-- imu -->
+     <link name="imu_link">
+        <visual>
+            <origin xyz="0.0 0.0 0.0" rpy="0.0 0.0 0.0"/>
+            <geometry>
+                <sphere radius="0.01"/>
+            </geometry>
+            <material name="red">
+                <color rgba="1.0 0.0 0.0 1.0"/>
+            </material>
+        </visual>
+     </link>
+     <joint name="joint_name" type="fixed">
+        <origin xyz="0.0 0.0 0.040" rpy="0.0 0.0 0.0"/>
+        <parent link="body"/>
+        <child link="imu_link"/>
+     </joint>
 </robot>

File: install/hexapod_description/share/hexapod_description/urdf/hexapod_gazebo.xacro (robot description, xacro)
@@ -85,4 +85,5 @@
                 <parameters>$(find hexapod_controller)/config/hexapod_controllers.yaml</parameters>
             </plugin>
+            <plugin filename="ignition-gazebo-imu-system" name="ignition::gazebo::systems::Imu"/>
         </xacro:if>
         <xacro:unless value="$(arg is_ignition)">
@@ -90,5 +91,37 @@
                 <parameters>$(find hexapod_controller)/config/hexapod_controllers.yaml</parameters>
             </plugin>
+            <plugin filename="gz-sim-imu-system" name="gz::sim::systems::Imu"/>
         </xacro:unless>
     </gazebo>
+    <gazebo reference="imu_link">
+        <sensor name="imu" type="imu">
+            <always_on>true</always_on>
+            <update_rate>100</update_rate>
+            <gz_frame_id>imu_link</gz_frame_id>
+            <topic>imu</topic>
+            <imu>
+                <!-- Orientation (roll, pitch, yaw) -->
+                <orientation>
+                    <noise type="gaussian">
+                        <mean>0.0</mean>
+                        <stddev>0.001</stddev> <!-- Adjust for orientation noise level -->
+                    </noise>
+                </orientation>
+                <!-- Angular Velocity (rate of rotation around each axis) -->
+                <angular_velocity>
+                    <noise type="gaussian">
+                        <mean>0.0</mean>
+                        <stddev>2e-4</stddev> <!-- Noise standard deviation for angular velocity -->
+                    </noise>
+                </angular_velocity>
+                <!-- Linear Acceleration (simulates linear velocity indirectly through integration) -->
+                <linear_acceleration>
+                    <noise type="gaussian">
+                        <mean>0.0</mean>
+                        <stddev>1.7e-2</stddev> <!-- Noise standard deviation for linear acceleration -->
+                    </noise>
+                </linear_acceleration>
+            </imu>
+        </sensor>
+    </gazebo>
 </robot>
